Commit message: aggiunta di nuove componenti nell urdf

File: urdf/arduinobot.urdf (robot description, URDF)
Before this commit: robot arduinobot, 1 links, 0 joints
Links:
- added link base_plate; visual mesh filename=package://simple_robot_arm/mesh/round_plate.STL scale=0.01 0.01 0.01
- added link base_plate_support; visual mesh filename=package://simple_robot_arm/mesh/plate.STL scale=0.01 0.01 0.01
Joints:
- added joint base_link_to_plate: type fixed, parent base_link, child base_plate, origin xyz=0 0 0.307
- added joint base_plate_to_support: type fixed, parent base_plate, child base_plate_support, origin xyz=0 0 0.05

Commit message: conclusione del modello urdf

File: urdf/arduinobot.urdf (robot description, URDF)
Before this commit: robot arduinobot, 3 links, 2 joints
Links:
- added link claw_support; visual mesh filename=package://simple_robot_arm/mesh/claw_support.STL scale=0.01 0.01 0.01
- added link forward_drive_arm; visual mesh filename=package://simple_robot_arm/mesh/forward_drive_arm.STL scale=0.01 0.01 0.01
- added link horizontal_arm; visual mesh filename=package://simple_robot_arm/mesh/horizontal_arm.STL scale=0.01 0.01 0.01
- added link left_finger; visual mesh filename=package://simple_robot_arm/mesh/left_finger.STL scale=0.01 0.01 0.01
- added link right_finger; visual mesh filename=package://simple_robot_arm/mesh/right_finger.STL scale=0.01 0.01 0.01
Joints:
- added joint base_support_to_forward_drive_arm: type revolute, parent base_plate_support, child forward_drive_arm, origin xyz=0 0 0.28, axis 1 0 0, limit lower=-1.57075 upper=1.57075 effort=1000.0 velocity=0.5
- added joint claw_support_to_left_finger: type revolute, parent claw_support, child left_finger, origin xyz=-0.215 0.16 -0.14, axis 0 0 1, limit lower=0 upper=1.57075 effort=1000.0 velocity=0.5
- added joint claw_support_to_right_finger: type revolute, parent claw_support, child right_finger, origin xyz=-0.035 0.16 -0.14, axis 0 0 1, limit lower=-1.57075 upper=0 effort=1000.0 velocity=0.5
- added joint forward_drive_arm_to_horizontal_arm: type revolute, parent forward_drive_arm, child horizontal_arm, origin xyz=0 0 0.8, axis 1 0 0, limit lower=-1.57075 upper=1.57075 effort=1000.0 velocity=0.5
- added joint horizontal_arm_to_claw_support: type fixed, parent horizontal_arm, child claw_support, origin xyz=0 0.82 0
- joint base_link_to_plate: axis (none) -> 0 0 1; limit (none) -> lower=0.0 upper=3.14 effort=1000.0 velocity=0.5; type fixed -> revolute

Commit message: utilizzo di arduino come subscriber per il movimento di un servpo

File: urdf/arduinobot.urdf (robot description, URDF)
Before this commit: robot arduinobot, 8 links, 7 joints
Links:
- removed link left_finger
- removed link right_finger
Joints:
- removed joint claw_support_to_left_finger
- removed joint claw_support_to_right_finger

Commit message: conclusione della comunicazione tra il braccio e ros

File: urdf/arduinobot.urdf (robot description, URDF)
Before this commit: robot arduinobot, 6 links, 5 joints
Joints:
- joint base_link_to_plate: limit lower=0.0 upper=3.14 effort=1000.0 velocity=0.5 -> lower=-1.57075 upper=1.57075 effort=1000.0 velocity=0.5

Commit message: lettura da joint states

File: urdf/arduinobot.urdf (robot description, URDF)
Before this commit: robot arduinobot, 6 links, 5 joints
Links:
- removed link base_plate_support
- added link tool_link
- added link world
- link base_link: geometry collision mesh filename=package://simple_robot_arm/mesh/basement.STL scale=0.01 0.01 0.01; visual mesh filename=package://simple_robot_arm/mesh/basement.STL scale=0.01 0.01 0.01
- link base_plate: geometry collision mesh filename=package://simple_robot_arm/mesh/round_plate.STL scale=0.01 0.01 0.01; visual mesh filename=package://simple_robot_arm/mesh/base_plate.STL scale=0.01 0.01 0.01
- link claw_support: geometry collision mesh filename=package://simple_robot_arm/mesh/claw_support.STL scale=0.01 0.01 0.01; visual mesh filename=package://simple_robot_arm/mesh/claw_support.STL scale=0.01 0.01 0.01
- link forward_drive_arm: geometry collision mesh filename=package://simple_robot_arm/mesh/forward_drive_arm.STL scale=0.01 0.01 0.01; visual mesh filename=package://simple_robot_arm/mesh/forward_drive_arm.STL scale=0.01 0.01 0.01
- link horizontal_arm: geometry collision mesh filename=package://simple_robot_arm/mesh/horizontal_arm.STL scale=0.01 0.01 0.01; visual mesh filename=package://simple_robot_arm/mesh/horizontal_arm.STL scale=0.01 0.01 0.01
Joints:
- removed joint base_link_to_plate
- removed joint base_plate_to_support
- removed joint base_support_to_forward_drive_arm
- removed joint forward_drive_arm_to_horizontal_arm
- added joint claw_support_to_tool: type fixed, parent claw_support, child tool_link, origin xyz=0 0 0
- added joint joint_1: type revolute, parent base_link, child base_plate, origin xyz=0 0 0.307, axis 0 0 1, limit lower=-1.5707963268 upper=1.5707963268 effort=1000.0 velocity=0.5
- added joint joint_2: type revolute, parent base_plate, child forward_drive_arm, origin xyz=0 0 0.28, axis 1 0 0, limit lower=-1.5707963268 upper=1.5707963268 effort=1000.0 velocity=0.5
- added joint joint_3: type revolute, parent forward_drive_arm, child horizontal_arm, origin xyz=0 0 0.8, axis 1 0 0, limit lower=-1.5707963268 upper=1.5707963268 effort=1000.0 velocity=0.5
- added joint joint_world: type fixed, parent world, child base_link, origin xyz=0 0 0 rpy=0 0 0

File: urdf/arduinobot.urdf.xacro (robot description, xacro)
@@ -119,3 +119,41 @@
         <origin xyz="0 0 0"/>
     </joint>
+    <!-- Transmissions-->
+    <transmission name="transmission_1">
+        <type>transmission_interface/SimpleTransmission</type>
+        <joint name="joint_1">
+            <hardwareInterface>PositionJointInterface</hardwareInterface>
+        </joint>
+        <actuator name="motor_1">
+            <hardwareInterface>PositionJointInterface</hardwareInterface>
+            <mechanicalReduction>1</mechanicalReduction>
+        </actuator>
+    </transmission>
+    <transmission name="transmission_2">
+        <type>transmission_interface/SimpleTransmission</type>
+        <joint name="joint_2">
+            <hardwareInterface>PositionJointInterface</hardwareInterface>
+        </joint>
+        <actuator name="motor_2">
+            <hardwareInterface>PositionJointInterface</hardwareInterface>
+            <mechanicalReduction>1</mechanicalReduction>
+        </actuator>
+    </transmission>
+    <transmission name="transmission_3">
+        <type>transmission_interface/SimpleTransmission</type>
+        <joint name="joint_3">
+            <hardwareInterface>PositionJointInterface</hardwareInterface>
+        </joint>
+        <actuator name="motor_3">
+            <hardwareInterface>PositionJointInterface</hardwareInterface>
+            <mechanicalReduction>1</mechanicalReduction>
+        </actuator>
+    </transmission>
+    <!-- Gazebo Configuration section -->
+    <gazebo>
+        <plugin name="gazebo_ros_control" filename="libgazebo_ros_control.so">
+            <robotNamespace>/arduinobot</robotNamespace>
+            <robotSimType>gazbo_roscontrol/DefaultRobotHWSim</robotSimType>
+        </plugin>
+    </gazebo>
 </robot>
